File: hardware/sesam_v2.brd (EAGLE design)
At the start: 70 x 70 mm, 11 parts, among them X2 C-GRID-06-70543

Commit message: minor changes
Routing:
- net N$4: track 41.9 -> 41.1 mm
- added copper zone on layer 16, net GND
Changed lines of the file:
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@@
 <wire x1="55.02" y1="7.46" x2="55.02" y2="5.46" width="0.3048" layer="16"/>
 <wire x1="55.02" y1="5.46" x2="54.98" y2="5.42" width="0.3048" layer="16"/>
-<wire x1="42.5" y1="46.98" x2="44.34" y2="49.84" width="0.3048" layer="16"/>
+<wire x1="42.5" y1="46.66" x2="44.34" y2="49.84" width="0.3048" layer="16"/>
 <wire x1="44.34" y1="49.84" x2="51.138" y2="49.84" width="0.3048" layer="16"/>
 <wire x1="51.138" y1="49.84" x2="51.212" y2="49.914" width="0.3048" layer="16"/>
@@
 <wire x1="51.22" y1="43.1" x2="51.22" y2="49.906" width="0.3048" layer="16"/>
 <wire x1="51.22" y1="49.906" x2="51.212" y2="49.914" width="0.3048" layer="16"/>
-<wire x1="42.5" y1="46.98" x2="42.5" y2="10.92" width="0.3048" layer="16"/>
-<wire x1="42.5" y1="10.92" x2="43.05" y2="10.37" width="0.3048" layer="16"/>
+<wire x1="42.5" y1="46.66" x2="42.5" y2="10.6" width="0.3048" layer="16"/>
+<wire x1="42.5" y1="10.6" x2="43.05" y2="10.37" width="0.3048" layer="16"/>
 </signal>
 <signal name="N$3">
@@
 <wire x1="13.64" y1="31.88" x2="11.13" y2="34.39" width="0.4064" layer="1"/>
 <wire x1="16.4" y1="5.1" x2="16.4" y2="3.8" width="0.3048" layer="1"/>
-<wire x1="16.4" y1="3.8" x2="15.46" y2="2.86" width="0.3048" layer="1"/>
-<wire x1="15.46" y1="2.86" x2="6.26" y2="2.86" width="0.3048" layer="1"/>
-<wire x1="6.26" y1="2.86" x2="4.72" y2="4.4" width="0.3048" layer="1"/>
+<wire x1="16.4" y1="3.8" x2="15.52" y2="3.1" width="0.3048" layer="1"/>
+<wire x1="15.52" y1="3.1" x2="5.9" y2="3.04" width="0.3048" layer="1"/>
+<wire x1="5.9" y1="3.04" x2="4.72" y2="4.4" width="0.3048" layer="1"/>
 <wire x1="4.72" y1="4.4" x2="4.72" y2="16.46" width="0.3048" layer="1"/>
 <wire x1="4.72" y1="16.46" x2="5.72" y2="17.46" width="0.3048" layer="1"/>
@@
 <wire x1="4" y1="19.15" x2="11.13" y2="19.15" width="0.4064" layer="1"/>
 <wire x1="18.96" y1="5.1" x2="18.96" y2="3.78" width="0.4064" layer="1"/>
-<wire x1="18.96" y1="3.78" x2="16.64" y2="1.46" width="0.4064" layer="1"/>
-<wire x1="16.64" y1="1.46" x2="5.72" y2="1.46" width="0.4064" layer="1"/>
-<wire x1="5.72" y1="1.46" x2="3.52" y2="3.66" width="0.4064" layer="1"/>
-<wire x1="3.52" y1="3.66" x2="3.52" y2="18.67" width="0.4064" layer="1"/>
+<wire x1="18.96" y1="3.78" x2="16.28" y2="2.06" width="0.4064" layer="1"/>
+<wire x1="16.28" y1="2.06" x2="5.36" y2="2.06" width="0.4064" layer="1"/>
+<wire x1="5.36" y1="2.06" x2="3.52" y2="4.04" width="0.4064" layer="1"/>
+<wire x1="3.52" y1="4.04" x2="3.52" y2="18.67" width="0.4064" layer="1"/>
 <wire x1="3.52" y1="18.67" x2="4" y2="19.15" width="0.4064" layer="1"/>
 </signal>
@@
 <vertex x="0" y="0"/>
 </polygon>
-<wire x1="51.212" y1="67.186" x2="63.974" y2="67.266" width="0.4064" layer="1"/>
-<wire x1="63.974" y1="67.266" x2="65.84" y2="65.4" width="0.4064" layer="1"/>
+<wire x1="51.212" y1="67.186" x2="65.854" y2="67.186" width="0.4064" layer="1"/>
+<wire x1="65.854" y1="67.186" x2="65.84" y2="65.4" width="0.4064" layer="1"/>
 <wire x1="45.969" y1="45.651" x2="45.92" y2="45.7" width="0.4064" layer="1"/>
-<wire x1="45.92" y1="45.7" x2="45.92" y2="61.974" width="0.4064" layer="1"/>
-<wire x1="45.92" y1="61.974" x2="51.212" y2="67.186" width="0.4064" layer="1"/>
+<wire x1="45.92" y1="45.7" x2="49.74" y2="61.614" width="0.4064" layer="1"/>
+<wire x1="49.74" y1="61.614" x2="51.212" y2="67.186" width="0.4064" layer="1"/>
 <wire x1="3.51" y1="21.69" x2="5.49" y2="21.69" width="0.4064" layer="1"/>
 <wire x1="5.49" y1="21.69" x2="6.98" y2="23.18" width="0.4064" layer="1"/>
@@
 <wire x1="45.92" y1="45.64" x2="45.969" y2="45.651" width="0.4064" layer="1"/>
 <wire x1="42.02" y1="37.9" x2="41.98" y2="34.64" width="0.4064" layer="1"/>
-<wire x1="41.98" y1="34.64" x2="41.42" y2="33.34" width="0.4064" layer="1"/>
-<wire x1="41.42" y1="33.34" x2="36.26" y2="33.26" width="0.4064" layer="1"/>
-<wire x1="36.26" y1="33.26" x2="35" y2="31.92" width="0.4064" layer="1"/>
+<wire x1="41.98" y1="34.64" x2="41.68" y2="33.22" width="0.4064" layer="1"/>
+<wire x1="41.68" y1="33.22" x2="36.26" y2="33.2" width="0.4064" layer="1"/>
+<wire x1="36.26" y1="33.2" x2="35" y2="31.92" width="0.4064" layer="1"/>
 <wire x1="22.3" y1="30.04" x2="22.3" y2="30.06" width="0.4064" layer="1"/>
 <wire x1="22.3" y1="30.06" x2="20.44" y2="31.92" width="0.4064" layer="1"/>
 <wire x1="20.44" y1="31.92" x2="20.5" y2="31.92" width="0.4064" layer="1"/>
 <wire x1="20.5" y1="31.92" x2="21.7" y2="33.12" width="0.4064" layer="1"/>
-<wire x1="21.7" y1="33.12" x2="27.16" y2="33.12" width="0.4064" layer="1"/>
-<wire x1="27.16" y1="33.12" x2="29.42" y2="35.38" width="0.4064" layer="1"/>
+<wire x1="21.7" y1="33.12" x2="27.44" y2="33.12" width="0.4064" layer="1"/>
+<wire x1="27.44" y1="33.12" x2="29.42" y2="35.38" width="0.4064" layer="1"/>
 <wire x1="29.42" y1="35.38" x2="29.42" y2="37.784646875" width="0.4064" layer="1"/>
 <wire x1="29.42" y1="37.784646875" x2="29.5610875" y2="37.925734375" width="0.4064" layer="1"/>
@@
 <wire x1="37.7" y1="5.32" x2="37.7" y2="16.78" width="0.3048" layer="16"/>
 <wire x1="37.7" y1="16.78" x2="32.7" y2="21.78" width="0.3048" layer="16"/>
-<wire x1="37.82" y1="5.35" x2="37.7" y2="5.32" width="0" layer="19" extent="1-16"/>
-<wire x1="32.47" y1="21.77" x2="32.7" y2="21.78" width="0" layer="19" extent="16-16"/>
+<polygon width="0.4064" layer="16" isolate="0.3048">
+<vertex x="0" y="70"/>
+<vertex x="70" y="70"/>
+<vertex x="70.02" y="39.84"/>
+<vertex x="60.06" y="39.84"/>
+<vertex x="60.06" y="18.32"/>
+<vertex x="70.08" y="18.32"/>
+<vertex x="70.08" y="-0.12"/>
+<vertex x="0.06" y="-0.12"/>
+<vertex x="0.06" y="69.96"/>
+</polygon>
 </signal>
 <signal name="N$13">
@@
 <wire x1="47.88" y1="3.6" x2="45.22" y2="0.94" width="0.3048" layer="1"/>
 <wire x1="45.22" y1="0.94" x2="17.78" y2="0.94" width="0.3048" layer="1"/>
-<wire x1="17.78" y1="0.94" x2="17.38" y2="0.54" width="0.3048" layer="1"/>
-<wire x1="17.38" y1="0.54" x2="5.4" y2="0.54" width="0.3048" layer="1"/>
-<wire x1="5.4" y1="0.54" x2="1.6" y2="4.34" width="0.3048" layer="1"/>
+<wire x1="17.78" y1="0.94" x2="17.2" y2="0.92" width="0.3048" layer="1"/>
+<wire x1="17.2" y1="0.92" x2="5.22" y2="0.92" width="0.3048" layer="1"/>
+<wire x1="5.22" y1="0.92" x2="1.6" y2="4.34" width="0.3048" layer="1"/>
 <wire x1="1.6" y1="4.34" x2="1.6" y2="19.66" width="0.3048" layer="1"/>
 <wire x1="1.6" y1="19.66" x2="2.46" y2="20.52" width="0.3048" layer="1"/>
@@
 <wire x1="52.89" y1="43.83" x2="51.48" y2="44.98" width="0.3048" layer="1"/>
 <wire x1="51.48" y1="44.98" x2="46.76" y2="44.98" width="0.3048" layer="1"/>
-<wire x1="46.76" y1="44.98" x2="42.96" y2="42.16" width="0.3048" layer="1"/>
-<wire x1="42.96" y1="42.16" x2="42.96" y2="35.04" width="0.3048" layer="1"/>
-<wire x1="42.96" y1="35.04" x2="42.56" y2="34.64" width="0.3048" layer="1"/>
-<wire x1="42.56" y1="34.64" x2="42.56" y2="26.18" width="0.3048" layer="1"/>
-<wire x1="42.56" y1="26.18" x2="41.76" y2="25.38" width="0.3048" layer="1"/>
-<wire x1="41.76" y1="25.38" x2="41.76" y2="23.44" width="0.3048" layer="1"/>
-<wire x1="41.76" y1="23.44" x2="40.09" y2="21.77" width="0.3048" layer="1"/>
+<wire x1="46.76" y1="44.98" x2="43.22" y2="42.4" width="0.3048" layer="1"/>
+<wire x1="43.22" y1="42.4" x2="43.22" y2="36.06" width="0.3048" layer="1"/>
+<wire x1="43.22" y1="36.06" x2="42.3" y2="32.88" width="0.3048" layer="1"/>
+<wire x1="42.3" y1="32.88" x2="42" y2="26.24" width="0.3048" layer="1"/>
+<wire x1="42" y1="26.24" x2="41.82" y2="25.38" width="0.3048" layer="1"/>
+<wire x1="41.82" y1="25.38" x2="41.82" y2="23.44" width="0.3048" layer="1"/>
+<wire x1="41.82" y1="23.44" x2="40.09" y2="21.77" width="0.3048" layer="1"/>
 </signal>
 <signal name="N$17">
 <contactref element="SERIAL" pad="1"/>
 <contactref element="U1" pad="TXD0"/>
-<wire x1="49.94" y1="18.54" x2="49.94" y2="31.1" width="0.3048" layer="1"/>
-<wire x1="49.94" y1="31.1" x2="53.88" y2="35.04" width="0.3048" layer="1"/>
+<wire x1="49.88" y1="18.74" x2="49.94" y2="31.3" width="0.3048" layer="1"/>
+<wire x1="49.94" y1="31.3" x2="53.88" y2="35.04" width="0.3048" layer="1"/>
 <wire x1="53.88" y1="35.04" x2="53.88" y2="44.64" width="0.3048" layer="1"/>
 <wire x1="53.88" y1="44.64" x2="57.431" y2="48.191" width="0.3048" layer="1"/>
-<wire x1="49.94" y1="18.54" x2="50.82" y2="17.66" width="0.3048" layer="1"/>
+<wire x1="49.88" y1="18.74" x2="50.82" y2="17.66" width="0.3048" layer="1"/>
 <wire x1="50.82" y1="17.66" x2="53.02" y2="17.66" width="0.3048" layer="1"/>
-<wire x1="53.02" y1="17.66" x2="53.94" y2="18.58" width="0.3048" layer="1"/>
-<wire x1="53.94" y1="18.58" x2="53.94" y2="22.9" width="0.3048" layer="1"/>
-<wire x1="53.94" y1="22.9" x2="55.02" y2="23.98" width="0.3048" layer="1"/>
+<wire x1="53.02" y1="17.66" x2="53.88" y2="18.52" width="0.3048" layer="1"/>
+<wire x1="53.88" y1="18.52" x2="53.88" y2="22.84" width="0.3048" layer="1"/>
+<wire x1="53.88" y1="22.84" x2="55.02" y2="23.98" width="0.3048" layer="1"/>
 <wire x1="55.02" y1="23.98" x2="59.28" y2="23.98" width="0.3048" layer="1"/>
 <wire x1="59.28" y1="23.98" x2="60.94" y2="22.32" width="0.3048" layer="1"/>
@@
 </signal>
 </signals>
+<errors>
+</errors>
 </board>
 </drawing>

Commit message: little changes
Connections:
- removed net N$23: U$1.IN-, X1.2
- net GND: now also U$1.IN-, X1.2
- net N$21: now also OLED.2
Routing:
- net N$21: track 28.6 -> 85.0 mm, vias 0 -> 1
- net GND: track 263.6 -> 300.2 mm
- net N$23: track 11.8 -> 0.00 mm
Changed lines of the file:
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@@
 <vertex x="0.06" y="69.96"/>
 </polygon>
+<contactref element="U$1" pad="IN-"/>
+<contactref element="X1" pad="2"/>
+<wire x1="4.395" y1="61.53" x2="9.37" y2="61.53" width="0.4064" layer="1"/>
+<wire x1="9.37" y1="61.53" x2="9.86" y2="62.02" width="0.4064" layer="1"/>
+<wire x1="9.86" y1="62.02" x2="9.98" y2="62.02" width="0.4064" layer="1"/>
+<wire x1="9.98" y1="62.02" x2="11.44" y2="63.48" width="0.4064" layer="1"/>
+<wire x1="11.44" y1="63.48" x2="11.44" y2="66.26" width="0.4064" layer="1"/>
+<wire x1="11.44" y1="66.26" x2="11.72" y2="66.54" width="0.4064" layer="1"/>
+<wire x1="11.72" y1="66.54" x2="11.72" y2="67.134" width="0.4064" layer="1"/>
+<wire x1="11.72" y1="67.134" x2="11.588" y2="67.186" width="0.4064" layer="1"/>
+<wire x1="32.7" y1="21.78" x2="32.47" y2="21.77" width="0" layer="19" extent="16-16"/>
+<wire x1="37.82" y1="5.35" x2="37.7" y2="5.32" width="0" layer="19" extent="1-16"/>
+<wire x1="4.395" y1="61.53" x2="1.78" y2="59.2" width="0.4064" layer="1"/>
+<wire x1="1.78" y1="59.2" x2="1.78" y2="39.08" width="0.4064" layer="1"/>
+<wire x1="1.78" y1="39.08" x2="2.32" y2="37.98" width="0.4064" layer="1"/>
 </signal>
 <signal name="N$13">
@@
 <wire x1="50.82" y1="24.26" x2="50.82" y2="20.97" width="0.3048" layer="1"/>
 <wire x1="50.82" y1="20.97" x2="50.89" y2="20.9" width="0.3048" layer="1"/>
+<contactref element="OLED" pad="2"/>
+<wire x1="42.76" y1="5.49" x2="42.76" y2="15.46" width="0.4064" layer="1"/>
+<wire x1="42.76" y1="15.46" x2="43.94" y2="16.64" width="0.4064" layer="1"/>
+<via x="43.94" y="16.64" extent="1-16" drill="0.6" shape="square"/>
+<wire x1="43.94" y1="16.64" x2="44" y2="39.34" width="0.4064" layer="16"/>
+<wire x1="44" y1="39.34" x2="43.5" y2="39.78" width="0.4064" layer="16"/>
+<wire x1="43.5" y1="39.78" x2="43.56" y2="42.38" width="0.4064" layer="16"/>
+<wire x1="43.56" y1="42.38" x2="44.58" y2="43" width="0.4064" layer="16"/>
+<wire x1="44.58" y1="43" x2="49.06" y2="43" width="0.4064" layer="16"/>
+<wire x1="49.06" y1="43" x2="50.52" y2="41.92" width="0.4064" layer="16"/>
+<wire x1="50.52" y1="41.92" x2="57.25796875" y2="42.2832375" width="0.4064" layer="16"/>
+<wire x1="57.25796875" y1="42.2832375" x2="59.971" y2="44.731" width="0.4064" layer="16"/>
+<wire x1="59.971" y1="44.731" x2="59.971" y2="45.651" width="0.4064" layer="16"/>
 </signal>
 <signal name="N$16">
@@
 <wire x1="4.445" y1="56.4" x2="4.395" y2="56.45" width="0.4064" layer="1"/>
 </signal>
-<signal name="N$23">
-<contactref element="U$1" pad="IN-"/>
-<contactref element="X1" pad="2"/>
-<wire x1="4.395" y1="61.53" x2="9.37" y2="61.53" width="0.4064" layer="1"/>
-<wire x1="9.37" y1="61.53" x2="9.86" y2="62.02" width="0.4064" layer="1"/>
-<wire x1="9.86" y1="62.02" x2="9.98" y2="62.02" width="0.4064" layer="1"/>
-<wire x1="9.98" y1="62.02" x2="11.44" y2="63.48" width="0.4064" layer="1"/>
-<wire x1="11.44" y1="63.48" x2="11.44" y2="66.26" width="0.4064" layer="1"/>
-<wire x1="11.44" y1="66.26" x2="11.72" y2="66.54" width="0.4064" layer="1"/>
-<wire x1="11.72" y1="66.54" x2="11.72" y2="67.134" width="0.4064" layer="1"/>
-<wire x1="11.72" y1="67.134" x2="11.588" y2="67.186" width="0.4064" layer="1"/>
-</signal>
 <signal name="N$6">

Commit message: new nice layout
Parts:
- moved X1 4.01 mm to (5.04, 63.0)
- moved OUTPUT_CON 2.52 mm to (25.3, 5.10)
- moved SERIAL 1.78 mm to (63.0, 46.6)
- moved RELAIS_3 1.07 mm to (35.3, 26.5)
- moved D1 0.95 mm to (66.8, 60.5)
- moved RELAIS_2 0.90 mm to (21.4, 26.5)
- moved U$1 0.68 mm to (31.5, 59.2)
- moved X2 0.57 mm to (59.2, 5.04)
- moved OLED 0.46 mm to (41.6, 5.04)
- moved RELAIS_1 0.39 mm to (7.56, 26.5)
- moved U1 0.35 mm to (55.4, 29.0)
Connections:
- net N$12: now also U1.ADC; no longer U1.GPIO9
Routing:
- net GND: track 300.2 -> 26.6 mm, vias 0 -> 1
- net N$13: track 108.6 -> 52.5 mm
- net N$14: track 82.1 -> 43.5 mm
- net N$16: track 94.3 -> 57.9 mm, vias 0 -> 1
- net N$21: track 85.0 -> 56.6 mm
- net N$17: track 51.4 -> 28.9 mm
- net 3V3: track 110.3 -> 127.5 mm, vias 1 -> 0
- net N$15: track 39.0 -> 26.1 mm
- net N$11: track 20.1 -> 32.4 mm
- net N$4: track 41.1 -> 52.5 mm
- net N$12: track 61.9 -> 53.8 mm
- net N$18: track 13.0 -> 20.8 mm
- net N$6: track 22.5 -> 27.4 mm
- net N$10: track 18.7 -> 23.1 mm
- net N$9: track 18.9 -> 22.1 mm
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
Commit message: ready for first board
Parts:
- RELAIS_1: value (none) -> V23100-V4005-A010
- RELAIS_2, RELAIS_3: value (none) -> V23100-A4005-A010
- renumbered U$1 to DC/DC, X1 to POWER, X2 to GPIO
Other:
- board text added: "esp8266-sesam"
- board text added: "https://hackerspace-bamberg.de/esp8266-sesam"
- board text added: "layout by xoquox"
