File: hardware/sesam_v2.brd (EAGLE design)
At the start: 70 x 70 mm, 11 parts

Commit message: nice new layout and board, better power supply added
Parts:
- removed D1: 3.3V, diode:DO35Z10
- added C1: 0.1µF, rcl:C0805
- added C2: 10µF, rcl:E2-5
- added IC1: 337T, linear:TO220H
Connections:
- net N$10 renamed GPIO5
- net N$12 renamed ADC
- net N$13 renamed GPIO13
- net N$14 renamed GPIO12
- net N$15 renamed GPIO14
- net N$17 renamed TX
- net N$19 renamed RST
- net N$20 renamed RX
- net N$9 renamed GPIO4
- removed net N$11: GPIO.3, U1.GPIO15
- removed net N$16: OLED.1, SERIAL.6, U1.GPIO0
- removed net N$18: SERIAL.3, U1.GPIO16
- removed net N$21: OLED.2, SERIAL.4, U1.GPIO2
- new net GPIO0: OLED.1, SERIAL.4, U1.GPIO0
- new net GPIO15: GPIO.3, SERIAL.6, U1.GPIO15
- new net GPIO16: U1.GPIO16
- new net GPIO2: OLED.2, SERIAL.3, U1.GPIO2
- new net POWER: C1.1, DC/DC.OUT+, IC1.3
- net 3V3: now also C2.+, IC1.2, U1.CH_PD; no longer D1.C, DC/DC.OUT+
- net GND: now also C1.2, C2.-, IC1.1; no longer D1.A
Routing:
- net GPIO15: track 0.00 -> 88.4 mm, vias 0 -> 1
- net GPIO2: track 0.00 -> 64.7 mm, vias 0 -> 1
- net N$16: track 57.9 -> 0.00 mm, vias 1 -> 0
- net N$21: track 56.6 -> 0.00 mm, vias 1 -> 0
- net GPIO0: track 0.00 -> 50.4 mm
- net N$11: track 32.4 -> 0.00 mm
- net GND: track 26.6 -> 0.00 mm, vias 1 -> 0
- net 3V3: track 127.5 -> 149.5 mm
- net N$18: track 20.5 -> 0.00 mm
- net TX: track 28.8 -> 42.2 mm
- net POWER: track 0.00 -> 8.91 mm
- net RX: track 34.8 -> 27.9 mm
- net ADC: track 53.8 -> 47.8 mm, vias 1 -> 0
- net N$13: track 27.4 -> 30.5 mm
- net GPIO12: track 43.4 -> 45.8 mm
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
Commit message: fixed power regulator
Parts:
- moved C2 24.6 mm to (44.2, 42.1), turned to 180 degrees
- moved C1 6.61 mm to (47.8, 55.5), turned to 90 degrees
Connections:
- net 3V3: now also IC1.3; no longer IC1.2
- net POWER: now also IC1.2; no longer IC1.3
Routing:
- net 3V3: track 149.5 -> 144.9 mm
- net POWER: track 8.91 -> 9.82 mm
Changed lines of the file:
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@@
 </element>
 <element name="IC1" library="linear" package="TO220H" value="337T" x="33.3375" y="54.2925" rot="MR270"/>
-<element name="C1" library="rcl" package="C0805" value="0.1µF" x="47.625" y="48.895" rot="R270"/>
-<element name="C2" library="rcl" package="E2-5" value="10µF" x="65.0875" y="55.245" rot="R90"/>
+<element name="C1" library="rcl" package="C0805" value="0.1µF" x="47.775" y="55.505" rot="R90"/>
+<element name="C2" library="rcl" package="E2-5" value="10µF" x="44.2375" y="42.145" rot="R180"/>
 </elements>
 <signals>
@@
 <contactref element="DC/DC" pad="OUT+"/>
 <contactref element="C1" pad="1"/>
-<contactref element="IC1" pad="3"/>
-<wire x1="51.312" y1="50.584" x2="48.364" y2="50.584" width="1.016" layer="1"/>
-<wire x1="48.364" y1="50.584" x2="47.625" y2="49.845" width="1.016" layer="1"/>
-<wire x1="47.625" y1="49.845" x2="45.405" y2="49.845" width="1.016" layer="1"/>
-<wire x1="45.405" y1="49.845" x2="43.4975" y2="51.7525" width="1.016" layer="1"/>
+<contactref element="IC1" pad="2"/>
+<wire x1="43.4975" y1="54.2925" x2="47.5125" y2="54.2925" width="1.016" layer="1"/>
+<wire x1="47.5125" y1="54.2925" x2="47.775" y2="54.555" width="1.016" layer="1"/>
+<wire x1="47.775" y1="54.555" x2="47.775" y2="54.121" width="1.016" layer="1"/>
+<wire x1="47.775" y1="54.121" x2="51.312" y2="50.584" width="1.016" layer="1"/>
 </signal>
 <signal name="3V3">
-<contactref element="IC1" pad="2"/>
 <contactref element="C2" pad="+"/>
 <contactref element="U1" pad="VCC"/>
@@
 <contactref element="U1" pad="CH_PD"/>
 <contactref element="SERIAL" pad="7"/>
-<wire x1="43.4975" y1="54.2925" x2="54.9275" y2="54.2925" width="1.016" layer="1"/>
-<wire x1="54.9275" y1="54.2925" x2="65.024" y2="54.2925" width="1.016" layer="1"/>
-<wire x1="65.024" y1="54.2925" x2="65.0875" y2="54.229" width="1.016" layer="1"/>
-<wire x1="47.24" y1="37.28" x2="47.24" y2="40.9575" width="1.016" layer="1"/>
-<wire x1="47.24" y1="40.9575" x2="47.24" y2="42.795" width="1.016" layer="1"/>
-<wire x1="47.24" y1="42.795" x2="51.1175" y2="46.6725" width="1.016" layer="1"/>
+<wire x1="47.24" y1="37.28" x2="47.19" y2="40.9575" width="1.016" layer="1"/>
+<wire x1="47.19" y1="40.9575" x2="47.22478125" y2="42.23571875" width="1.016" layer="1"/>
+<wire x1="47.22478125" y1="42.23571875" x2="47.24" y2="42.795" width="1.016" layer="1"/>
+<wire x1="47.24" y1="42.795" x2="50.0725" y2="45.6275" width="1.016" layer="1"/>
+<wire x1="50.0725" y1="45.6275" x2="51.1175" y2="46.6725" width="1.016" layer="1"/>
 <wire x1="51.1175" y1="46.6725" x2="53.34" y2="46.6725" width="1.016" layer="1"/>
 <wire x1="53.34" y1="46.6725" x2="55.245" y2="48.5775" width="1.016" layer="1"/>
-<wire x1="55.245" y1="48.5775" x2="55.245" y2="53.975" width="1.016" layer="1"/>
-<wire x1="55.245" y1="53.975" x2="54.9275" y2="54.2925" width="1.016" layer="1"/>
-<wire x1="66.81" y1="47.89" x2="66.81" y2="52.5065" width="1.016" layer="1"/>
-<wire x1="66.81" y1="52.5065" x2="65.0875" y2="54.229" width="1.016" layer="1"/>
 <wire x1="57.24" y1="37.28" x2="57.24" y2="39.915" width="0.254" layer="1"/>
 <wire x1="57.24" y1="39.915" x2="56.1975" y2="40.9575" width="0.254" layer="1"/>
-<wire x1="56.1975" y1="40.9575" x2="47.24" y2="40.9575" width="0.254" layer="1"/>
+<wire x1="56.1975" y1="40.9575" x2="47.19" y2="40.9575" width="0.254" layer="1"/>
 <wire x1="40.31" y1="5.04" x2="40.31" y2="3.505" width="0.8128" layer="1"/>
 <wire x1="40.31" y1="3.505" x2="42.2275" y2="1.5875" width="0.8128" layer="1"/>
@@
 <wire x1="55.41" y1="5.04" x2="55.41" y2="2.0575" width="0.8128" layer="1"/>
 <wire x1="55.41" y1="2.0575" x2="55.88" y2="1.5875" width="0.8128" layer="1"/>
-<wire x1="66.81" y1="47.89" x2="68.3975" y2="47.89" width="0.8128" layer="1"/>
+<wire x1="66.81" y1="47.89" x2="67.5" y2="47.89" width="0.8128" layer="1"/>
+<wire x1="67.5" y1="47.89" x2="68.3975" y2="47.89" width="0.8128" layer="1"/>
 <wire x1="68.3975" y1="47.89" x2="69.5325" y2="46.755" width="0.8128" layer="1"/>
+<contactref element="IC1" pad="3"/>
+<wire x1="43.4975" y1="51.7525" x2="43.9475" y2="51.7525" width="1.016" layer="1"/>
+<wire x1="43.9475" y1="51.7525" x2="50.0725" y2="45.6275" width="1.016" layer="1"/>
+<wire x1="55.245" y1="48.5775" x2="55.245" y2="51.295" width="1.016" layer="1"/>
+<wire x1="55.245" y1="51.295" x2="56.4" y2="52.45" width="1.016" layer="1"/>
+<wire x1="56.4" y1="52.45" x2="65.3" y2="52.45" width="1.016" layer="1"/>
+<wire x1="65.3" y1="52.45" x2="66.7" y2="51.05" width="1.016" layer="1"/>
+<wire x1="66.7" y1="51.05" x2="66.7" y2="48.69" width="1.016" layer="1"/>
+<wire x1="66.7" y1="48.69" x2="67.5" y2="47.89" width="1.016" layer="1"/>
+<wire x1="45.2535" y1="42.145" x2="47.1340625" y2="42.145" width="1.016" layer="1"/>
+<wire x1="47.1340625" y1="42.145" x2="47.22478125" y2="42.23571875" width="1.016" layer="1"/>
 </signal>
 <signal name="N$3">

Commit message: some layout tweeks
Parts:
- renumbered OUTPUT_CON to RELAYS_CON
Routing:
- net N$7: track 0.00 -> 9.59 mm
- net N$8: track 0.00 -> 2.74 mm
- net N$6: track 0.00 -> 2.65 mm
- net 3V3: track 144.9 -> 144.1 mm

Commit message: fixed GND connections
Routing:
- net GND: track 0.00 -> 15.0 mm
- net N$7: track 9.59 -> 0.00 mm
- net N$8: track 2.74 -> 0.00 mm
- net N$6: track 2.65 -> 0.00 mm
Changed lines of the file:
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@@
 <?xml version="1.0" encoding="utf-8"?>
 <!DOCTYPE eagle SYSTEM "eagle.dtd">
-<eagle version="6.6.0">
+<eagle version="7.6.0">
 <drawing>
 <settings>
@@
 <pass name="Default">
 <param name="RoutingGrid" value="50mil"/>
+<param name="AutoGrid" value="1"/>
+<param name="Efforts" value="0"/>
+<param name="TopRouterVariant" value="1"/>
 <param name="tpViaShape" value="round"/>
 <param name="PrefDir.1" value="/"/>
@@
 <contactref element="GPIO" pad="6"/>
 <contactref element="SERIAL" pad="2"/>
+<wire x1="17.05" y1="8.45" x2="20.8" y2="8.45" width="0.4064" layer="1"/>
+<wire x1="20.8" y1="8.45" x2="22.75" y2="6.6" width="0.4064" layer="1"/>
+<wire x1="22.75" y1="6.6" x2="22.75" y2="3.7" width="0.4064" layer="1"/>
+<wire x1="22.75" y1="3.7" x2="22.95" y2="3.55" width="0.254" layer="1"/>
+<wire x1="27.85" y1="6.35" x2="27.85" y2="3.7" width="0.4064" layer="1"/>
+<wire x1="41.6" y1="3.85" x2="41.6" y2="6.45" width="0.4064" layer="1"/>
+<wire x1="41.6" y1="6.45" x2="41.5" y2="6.55" width="0.254" layer="1"/>
+<wire x1="37.77" y1="5.04" x2="41.6" y2="3.85" width="0" layer="19" extent="1-1"/>
 </signal>
 <signal name="N$1">
@@
 <wire x1="60.6425" y1="5.1925" x2="60.49" y2="5.04" width="0.254" layer="16"/>
 </signal>
-<signal name="N$6">
-<wire x1="27.85" y1="6.35" x2="27.85" y2="3.7" width="0.4064" layer="1"/>
-</signal>
-<signal name="N$7">
-<wire x1="17.05" y1="8.45" x2="20.8" y2="8.45" width="0.4064" layer="1"/>
-<wire x1="20.8" y1="8.45" x2="22.75" y2="6.6" width="0.4064" layer="1"/>
-<wire x1="22.75" y1="6.6" x2="22.75" y2="3.7" width="0.4064" layer="1"/>
-<wire x1="22.75" y1="3.7" x2="22.95" y2="3.55" width="0.254" layer="1"/>
-</signal>
-<signal name="N$8">
-<wire x1="41.6" y1="3.85" x2="41.6" y2="6.45" width="0.4064" layer="1"/>
-<wire x1="41.6" y1="6.45" x2="41.5" y2="6.55" width="0.254" layer="1"/>
-</signal>
 </signals>
